Commit message: [ADD]: added model loader and model files

File: res/templates/urdf/r2d2.urdf (robot description, URDF)
Before this commit: robot physics, 16 links, 15 joints
Links:
- link left_gripper: geometry collision mesh filename=r2d2_meshes/l_finger.stl; visual mesh filename=r2d2_meshes/l_finger.stl
- link left_tip: geometry collision mesh filename=r2d2_meshes/l_finger_tip.stl; visual mesh filename=r2d2_meshes/l_finger_tip.stl
- link right_gripper: geometry collision mesh filename=r2d2_meshes/l_finger.stl; visual mesh filename=r2d2_meshes/l_finger.stl
- link right_tip: geometry collision mesh filename=r2d2_meshes/l_finger_tip.stl; visual mesh filename=r2d2_meshes/l_finger_tip.stl
