Commit message: [Updated]: walker-2d urdf model for raisim-tests
Changes:

* Added a full walker2d model for tests using raisim

File: res/xml/tests/raisim/walker.urdf (robot description, URDF)
Before this commit: robot walker, 7 links, 6 joints
Links:
- added link left_foot, mass 1; collision capsule length=0.2 radius=0.05; visual capsule length=0.2 radius=0.05
- added link left_leg, mass 1; collision capsule length=0.50 radius=0.04; visual capsule length=0.50 radius=0.04
- added link right_foot, mass 1; collision capsule length=0.2 radius=0.05; visual capsule length=0.2 radius=0.05
- added link right_leg, mass 1; collision capsule length=0.50 radius=0.04; visual capsule length=0.50 radius=0.04
- link left_thigh: geometry collision capsule length=0.45 radius=0.05; visual capsule length=0.45 radius=0.05
- link right_thigh: geometry collision capsule length=0.45 radius=0.05; visual capsule length=0.45 radius=0.05
- link torso: geometry collision capsule length=0.6 radius=0.07; visual capsule length=0.6 radius=0.07
Joints:
- removed joint plane_z
- added joint left_ankle: type revolute, parent left_leg, child left_foot, origin xyz=0.0 0.0 -0.5, axis 0 1 0
- added joint left_knee: type revolute, parent left_thigh, child left_leg, origin xyz=0.0 0.0 -0.45, axis 0 1 0
- added joint ref_world: type fixed, parent world, child reference_1
- added joint right_ankle: type revolute, parent right_leg, child right_foot, origin xyz=0.0 0.0 -0.5, axis 0 1 0
- added joint right_knee: type revolute, parent right_thigh, child right_leg, origin xyz=0.0 0.0 -0.45, axis 0 1 0
- joint ref_plane_x: child reference_1 -> reference_2; parent world -> reference_1; type fixed -> prismatic
- joint ref_plane_z: axis 1 0 0 -> 0 0 1; child reference_2 -> reference_3; parent reference_1 -> reference_2
- joint ref_rot_y: axis 0 0 1 -> 0 1 0; child reference_3 -> torso; parent reference_2 -> reference_3; type prismatic -> revolute
